Commit message: Se simplificaron las coliciones en las llantas

File: MovilOmnidireccional_description/urdf/yahboomcar_X3.urdf (robot description, URDF)
Before this commit: robot yahboomcar_X3, 9 links, 8 joints
Links:
- link back_left_wheel: geometry collision cylinder length=0.030 radius=0.0325; visual mesh filename=package://MovilOmnidireccional_description/meshes/X3/back_l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
- link back_right_wheel: geometry collision cylinder length=0.030 radius=0.0325; visual mesh filename=package://MovilOmnidireccional_description/meshes/X3/back_r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
- link front_left_wheel: geometry collision cylinder length=0.030 radius=0.0325; visual mesh filename=package://MovilOmnidireccional_description/meshes/X3/front_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
- link front_right_wheel: geometry collision cylinder length=0.030 radius=0.0325; visual mesh filename=package://MovilOmnidireccional_description/meshes/X3/front_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
