Commit message: Se modifico la colision del carrito a primitivas para simplificar el funcionamiento

File: MovilOmnidireccional_description/urdf/lidar.xacro (robot description, xacro)
@@ -11,5 +11,5 @@
             <collision>
                 <geometry>
-                    <cylinder radius="0.1" length="0.05" />
+                    <cylinder radius="0.05" length="0.05" />
                 </geometry>
                     <origin xyz="0 0 0" rpy="0 0 0" />

File: MovilOmnidireccional_description/urdf/yahboomcar_X3.urdf (robot description, URDF)
Before this commit: robot yahboomcar_X3, 9 links, 8 joints
Links:
- link base_link: geometry collision box size=0.24 0.135 0.0735; visual mesh filename=package://MovilOmnidireccional_description/meshes/X3/base_l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

Commit message: Se quito el lidar duplicado

File: MovilOmnidireccional_description/urdf/lidar.xacro (robot description, xacro)
@@ -1,5 +1,5 @@
 <?xml version="1.0"?>
 <robot name="omnidirectional" xmlns:xacro="http://ros.org/wiki/xacro" >
-    <link name="lidar_link">
+   <!-- <link name="lidar_link">
             <visual>
                 <geometry>
@@ -22,17 +22,17 @@
                         izz="0.1" />
             </inertial>
-    </link>
+    </link> -->
     <link name="lidar_sensor" />
-    <joint name="lidar_joint" type="fixed" >
+   <!-- <joint name="lidar_joint" type="fixed" >
         <parent link="base_link" />
-        <child link="lidar_link" />
+        <child link="laser_link" />
         <origin xyz="0 0 0.075" rpy="0 0 0" />
-    </joint>
+    </joint> -->
     <joint name="lidar_sensor_joint" type="fixed" >
-        <parent link="lidar_link" />
+        <parent link="laser_link" />
         <child link="lidar_sensor" />
         <origin xyz="0 0 0" rpy="0 0 0" />
     </joint>
-    <gazebo reference="lidar_link" >
+    <gazebo reference="laser_link" >
         <material>Gazebo/Blue</material>
     </gazebo>
