Commit message: Intento de visualizar en gz, NO FUNCIONA,Error en el controlador de velocidad

File: MovilOmnidireccional_description/urdf/omnidirectional_X3_controler.xacro (robot description, xacro)
@@ -3,8 +3,8 @@
     <xacro:property name="package_name" value="MovilOmnidireccional_description"/>
     <xacro:include filename="$(find ${package_name})/urdf/omnidirectional_X3.urdf"/>
+    <xacro:include filename="$(find ${package_name})/urdf/omnidirectional_gz_propierties.xacro"/>
+    <xacro:include filename="$(find ${package_name})/urdf/omnidirectional_control.xacro"/>
     <xacro:include filename="$(find ${package_name})/urdf/lidar.xacro"/>
     <xacro:include filename="$(find ${package_name})/urdf/camera.xacro"/>
     <xacro:include filename="$(find ${package_name})/urdf/imu.xacro"/>
-    <xacro:include filename="$(find ${package_name})/urdf/omnidirectional_gz_propierties.xacro"/>
-    <xacro:include filename="$(find ${package_name})/urdf/omnidirectional_control.xacro"/>
 </robot>

File: MovilOmnidireccional_description/urdf/omnidirectional_control.xacro (robot description, xacro)
@@ -13,5 +13,5 @@
         </plugin>
     </gazebo>
-  <!-- THIS PLUGIN IS USED TO CORRECTLY VISUALIZED JOINTS POSITION ON RVIZ  -->
+  <!-- THIS PLUGIN IS USED TO CORRECTLY VISUALIZED JOINTS POSITION ON RVIZ   -->
     <gazebo>
         <plugin name="joint_states_gz" filename="libgazebo_ros_joint_state_publisher.so">
@@ -20,8 +20,8 @@
         </ros>
         <update_rate>30</update_rate>
-        <joint_name>wheel_left_front_joint</joint_name>
-        <joint_name>wheel_rigth_front_joint</joint_name>
-        <joint_name>wheel_left_back_joint</joint_name>
-        <joint_name>wheel_rigth_back_joint</joint_name>
+        <joint_name>front_right_joint</joint_name>
+        <joint_name>front_left_joint</joint_name>
+        <joint_name>back_right_joint</joint_name>
+        <joint_name>back_left_joint</joint_name>
         </plugin>
     </gazebo>
@@ -31,6 +31,6 @@
             <plugin>gazebo_ros2_control/GazeboSystem</plugin>
         </hardware>
-    <!--List of joints to be controlled -->
-        <joint name="wheel_left_front_joint">
+    <!--List of joints to be controlled  -->
+        <joint name="front_right_joint">
             <command_interface name="velocity"/>
             <state_interface name="position"/>
@@ -38,5 +38,5 @@
             <state_interface name="effort"/>
         </joint>
-        <joint name="wheel_rigth_front_joint">
+        <joint name="front_left_joint">
             <command_interface name="velocity"/>
             <state_interface name="position"/>
@@ -44,5 +44,5 @@
             <state_interface name="effort"/>
         </joint>
-        <joint name="wheel_left_back_joint">
+        <joint name="back_right_joint">
             <command_interface name="velocity"/>
             <state_interface name="position"/>
@@ -50,5 +50,5 @@
             <state_interface name="effort"/>
         </joint>
-        <joint name="wheel_rigth_back_joint">
+        <joint name="back_left_joint">
             <command_interface name="velocity"/>
             <state_interface name="position"/>
